File: Hardware/LoRa_beacons_receiver/LoRa_beacons_receiver.kicad_pcb (KiCad board)
At the start: 2 copper layers, 65 x 53 mm, 44 parts, among them J1 Conn_Coaxial, J2 USB_C_Receptacle_USB2.0_16P, J3 I2C_Display, J4 ST-Link, J5 1PPS_out, J6 Conn_02x09_Counter_Clockwise, SW1 RST_button, SW2 BOOT_button, U1 Wio-E5, U2 CP2102N-Axx-xQFN28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

Commit message: Minor PCB changes
Routing:
- net /RST: track 87.2 -> 86.5 mm
- net UART1_RX-USB_TX: track 11.9 -> 12.4 mm
- net GND: vias 87 -> 86
