File: Hardware/LoRa_beacons_receiver/LoRa_beacons_receiver.kicad_pcb (KiCad board)
At the start: 2 copper layers, 65 x 53 mm, 44 parts, among them J1 Conn_Coaxial, J2 USB_C_Receptacle_USB2.0_16P, J3 I2C_Display, J4 ST-Link, J5 1PPS_out, J6 Conn_02x09_Counter_Clockwise, SW1 RST_button, SW2 BOOT_button, U1 Wio-E5, U2 CP2102N-Axx-xQFN28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

Commit message: fix: repetitive beacon reception; basic 1PPS (WIP); hw: final changes before PSB order
Parts:
- F1: footprint Fuse:Fuse_0805_2012Metric_Pad1.15x1.40mm_HandSolder -> Fuse:Fuse_0603_1608Metric_Pad1.05x0.95mm_HandSolder
- moved F1 0.10 mm to (109.5, 65.1)
