File: Hardware/LoRa_beacons_receiver/LoRa_beacons_receiver.kicad_sch (KiCad schematic)
At the start: 44 parts, among them J1 Conn_Coaxial, J2 USB_C_Receptacle_USB2.0_16P, J3 I2C_Display, J4 ST-Link, J5 1PPS_out, J6 Conn_02x09_Counter_Clockwise, SW1 RST_button, SW2 BOOT_button, U1 Wio-E5, U2 CP2102N-Axx-xQFN28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

Commit message: fix: repetitive beacon reception; basic 1PPS (WIP); hw: final changes before PSB order
Parts:
- C1, C10, C3, C6, C8: Manufacturer part number (none) -> 08055C104JAT2A
- C2, C5, C7: Manufacturer part number (none) -> CC0805KKX7R7BB105
- C4: Manufacturer part number (none) -> TMK212AB7475KG-T
- D1: Manufacturer part number (none) -> SP0503BAHTG-LF
- D2, D4, D5, D6: Manufacturer part number (none) -> LTST-C171KRKT
- D3: Manufacturer part number (none) -> MBR130LSFT1G
- F1: footprint Fuse:Fuse_0805_2012Metric_Pad1.15x1.40mm_HandSolder -> Fuse:Fuse_0603_1608Metric_Pad1.05x0.95mm_HandSolder; Manufacturer part number (none) -> ERBRE1R00V
- H1, H2, H3, H4, J3, U1: Manufacturer part number (none) -> -
- J1: Manufacturer part number (none) -> RF2-143-T-17-50-G
- J2: Manufacturer part number (none) -> USB4105-GF-A-120
- J4: Manufacturer part number (none) -> ZL262-5SG
- J5: Manufacturer part number (none) -> ZL263-2SG
- J6: Manufacturer part number (none) -> ZL262-9SG
- R1, R2: Manufacturer part number (none) -> WR08X5101FTL
- R10, R7, R8, R9: value 56R -> 100R; Manufacturer part number (none) -> CRCW0805100RFKTABC
- R11, R12, R3: Manufacturer part number (none) -> CRCW08054K70FKTABC
- R4, R5: Manufacturer part number (none) -> CRGH0805J22R
- R6: Manufacturer part number (none) -> ERJP06J471V
- SW1, SW2: Manufacturer part number (none) -> TACT4101-11250-A
- U2: Manufacturer part number (none) -> CP2102-GM
- U3: Manufacturer part number (none) -> AP2112K-3.3TRG1
- U5: Manufacturer part number (none) -> 74LVC1G17GV.125

Commit message: WIP
Other:
- title: (none) -> LoRaWAN Class-B beacons receiver
Changed lines of the file:
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@@
 	(generator_version "9.0")
 	(paper "A3")
+	(title_block
+		(title "LoRaWAN Class-B beacons receiver")
+		(date "2026-02-26")
+		(rev "A")
+	)
 	(rectangle
 		(start 101.6 220.98)
@@
 		)
 	)
-	(text_box "Poznamky\n"
-		(exclude_from_sim no)
-		(at 358.14 15.24 0)
-		(size 45.72 20.32)
-		(margins 0.9525 0.9525 0.9525 0.9525)
-		(stroke
-			(width 0)
-			(type solid)
-		)
-		(fill
-			(type none)
-		)
-		(effects
-			(font
-				(size 1.27 1.27)
-				(thickness 0.254)
-				(bold yes)
-			)
-			(justify left top)
-		)
-	)
